File: camera_controller/camera_controller_2.kicad_sch (KiCad schematic)
At the start: 31 parts, among them Q3 ZXTC2045E6TA, Q4 ZXTC2045E6TA, Q5 ZXTC2045E6TA, U5 ADS1115IDGS, U7 HMHA2801, U8 MAX3232EIDWR

Commit message: Removed neopixel status led and restored dual red/green status led support.
Minor tweaks to RTO pinouts.
Parts:
- C10: value 1uF -> 1 uF
Changed lines of the file:
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@@
 			)
 		)
-		(property "Value" "1uF"
+		(property "Value" "1 uF"
 			(at 219.71 44.958 0)
 			(effects
