File: remote_turn_on/remote_turn_on.kicad_pcb (KiCad board)
At the start: 4 copper layers, 20 x 25 mm, 15 parts, among them J1 SM08B-NSHSS-TB LFSN, U1 ATtiny85-20S, U2 MLX92231LSE

Commit message: Removed neopixel status led and restored dual red/green status led support.
Minor tweaks to RTO pinouts.
Parts:
- R1, R4: value 200 -> 220
- U2: value MLX92231LSE -> MLX92231LSE-AAA-009
Connections:
- D1 pad 1: Cam Status + -> Cam Status -
- D1 pad 2: Cam Status - -> Cam Status +
- J1 pad 7: Cam Status + -> Cam Status -
- J1 pad 8: Cam Status - -> Cam Status +
Routing:
- net Cam Status -: track 6.95 -> 10.8 mm
- net Cam Status +: track 10.8 -> 6.95 mm
Changed lines of the file:
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@@
 			(size 0.6604 1.7018)
 			(layers "F.Cu" "F.Mask" "F.Paste")
-			(net 4 "Cam Status +")
+			(net 3 "Cam Status -")
 			(pinfunction "7")
 			(pintype "unspecified")
@@
 			(size 0.6604 1.7018)
 			(layers "F.Cu" "F.Mask" "F.Paste")
-			(net 3 "Cam Status -")
+			(net 4 "Cam Status +")
 			(pinfunction "8")
 			(pintype "unspecified")
@@
 			(layers "F.Cu" "F.Mask" "F.Paste")
 			(roundrect_rratio 0.2)
-			(net 4 "Cam Status +")
+			(net 3 "Cam Status -")
 			(pinfunction "KA")
 			(pintype "input")
@@
 			(layers "F.Cu" "F.Mask" "F.Paste")
 			(roundrect_rratio 0.2)
-			(net 3 "Cam Status -")
+			(net 4 "Cam Status +")
 			(pinfunction "AK")
 			(pintype "input")
@@
 			)
 		)
-		(property "Value" "MLX92231LSE"
+		(property "Value" "MLX92231LSE-AAA-009"
 			(at 0 2.4 90)
 			(layer "F.Fab")
@@
 			)
 		)
-		(property "Value" "200"
+		(property "Value" "220"
 			(at 0 -1.65 0)
 			(layer "B.Fab")
@@
 			)
 		)
-		(property "Value" "200"
+		(property "Value" "220"
 			(at 0 -1.65 0)
 			(layer "B.Fab")
@@
 	)
 	(segment
-		(start 75.6 62.7)
-		(end 76 62.3)
+		(start 77.5 68.080363)
+		(end 77.1312 68.449163)
 		(width 0.2)
 		(layer "F.Cu")
@@
 	)
 	(segment
-		(start 76 62.3)
-		(end 76 61.3)
+		(start 73.2 65.780363)
+		(end 73.2 61.3)
 		(width 0.2)
 		(layer "F.Cu")
@@
 	)
 	(segment
-		(start 76.5 67.297263)
-		(end 75.797263 67.297263)
+		(start 77.1312 68.449163)
+		(end 75.8688 68.449163)
 		(width 0.2)
 		(layer "F.Cu")
@@
 	)
 	(segment
-		(start 75.797263 67.297263)
-		(end 75.6 67.1)
+		(start 77.5 67.297263)
+		(end 77.5 68.080363)
 		(width 0.2)
 		(layer "F.Cu")
@@
 	)
 	(segment
-		(start 75.6 67.1)
-		(end 75.6 62.7)
+		(start 75.8688 68.449163)
+		(end 73.2 65.780363)
 		(width 0.2)
 		(layer "F.Cu")
@@
 	)
 	(segment
-		(start 77.5 68.080363)
-		(end 77.1312 68.449163)
+		(start 75.6 62.7)
+		(end 76 62.3)
 		(width 0.2)
 		(layer "F.Cu")
@@
 	)
 	(segment
-		(start 73.2 65.780363)
-		(end 73.2 61.3)
+		(start 76 62.3)
+		(end 76 61.3)
 		(width 0.2)
 		(layer "F.Cu")
@@
 	)
 	(segment
-		(start 77.1312 68.449163)
-		(end 75.8688 68.449163)
+		(start 76.5 67.297263)
+		(end 75.797263 67.297263)
 		(width 0.2)
 		(layer "F.Cu")
@@
 	)
 	(segment
-		(start 77.5 67.297263)
-		(end 77.5 68.080363)
+		(start 75.797263 67.297263)
+		(end 75.6 67.1)
 		(width 0.2)
 		(layer "F.Cu")
@@
 	)
 	(segment
-		(start 75.8688 68.449163)
-		(end 73.2 65.780363)
+		(start 75.6 67.1)
+		(end 75.6 62.7)
 		(width 0.2)
 		(layer "F.Cu")

Commit message: Minor updates to controller, 3rd stab at hadron breakout
Minor updates to controller and firmware to make labels more consistent. Took another try at the hadron IO breakout. Old manufacture files removed.
Connections:
- net Cam Status + renamed Cam Status R
- net Cam Status - renamed Cam Status G
Changed lines of the file:
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@@
 	(net 1 "3.3v")
 	(net 2 "GND")
-	(net 3 "Cam Status -")
-	(net 4 "Cam Status +")
+	(net 3 "Cam Status R")
+	(net 4 "Cam Status G")
 	(net 5 "Net-(D2-Pad2)")
 	(net 6 "Net-(D2-Pad1)")
@@
 			(size 0.6604 1.7018)
 			(layers "F.Cu" "F.Mask" "F.Paste")
-			(net 3 "Cam Status -")
+			(net 4 "Cam Status G")
 			(pinfunction "7")
 			(pintype "unspecified")
@@
 			(size 0.6604 1.7018)
 			(layers "F.Cu" "F.Mask" "F.Paste")
-			(net 4 "Cam Status +")
+			(net 3 "Cam Status R")
 			(pinfunction "8")
 			(pintype "unspecified")
@@
 			(layers "F.Cu" "F.Mask" "F.Paste")
 			(roundrect_rratio 0.2)
-			(net 3 "Cam Status -")
+			(net 4 "Cam Status G")
 			(pinfunction "KA")
 			(pintype "input")
@@
 			(layers "F.Cu" "F.Mask" "F.Paste")
 			(roundrect_rratio 0.2)
-			(net 4 "Cam Status +")
+			(net 3 "Cam Status R")
 			(pinfunction "AK")
 			(pintype "input")
@@
 	)
 	(segment
-		(start 77.5 68.080363)
-		(end 77.1312 68.449163)
+		(start 75.6 62.7)
+		(end 76 62.3)
 		(width 0.2)
 		(layer "F.Cu")
@@
 	)
 	(segment
-		(start 73.2 65.780363)
-		(end 73.2 61.3)
+		(start 76 62.3)
+		(end 76 61.3)
 		(width 0.2)
 		(layer "F.Cu")
@@
 	)
 	(segment
-		(start 77.1312 68.449163)
-		(end 75.8688 68.449163)
+		(start 76.5 67.297263)
+		(end 75.797263 67.297263)
 		(width 0.2)
 		(layer "F.Cu")
@@
 	)
 	(segment
-		(start 77.5 67.297263)
-		(end 77.5 68.080363)
+		(start 75.797263 67.297263)
+		(end 75.6 67.1)
 		(width 0.2)
 		(layer "F.Cu")
@@
 	)
 	(segment
-		(start 75.8688 68.449163)
-		(end 73.2 65.780363)
+		(start 75.6 67.1)
+		(end 75.6 62.7)
 		(width 0.2)
 		(layer "F.Cu")
@@
 	)
 	(segment
-		(start 75.6 62.7)
-		(end 76 62.3)
+		(start 77.5 68.080363)
+		(end 77.1312 68.449163)
 		(width 0.2)
 		(layer "F.Cu")
@@
 	)
 	(segment
-		(start 76 62.3)
-		(end 76 61.3)
+		(start 73.2 65.780363)
+		(end 73.2 61.3)
 		(width 0.2)
 		(layer "F.Cu")
@@
 	)
 	(segment
-		(start 76.5 67.297263)
-		(end 75.797263 67.297263)
+		(start 77.1312 68.449163)
+		(end 75.8688 68.449163)
 		(width 0.2)
 		(layer "F.Cu")
@@
 	)
 	(segment
-		(start 75.797263 67.297263)
-		(end 75.6 67.1)
+		(start 77.5 67.297263)
+		(end 77.5 68.080363)
 		(width 0.2)
 		(layer "F.Cu")
@@
 	)
 	(segment
-		(start 75.6 67.1)
-		(end 75.6 62.7)
+		(start 75.8688 68.449163)
+		(end 73.2 65.780363)
 		(width 0.2)
 		(layer "F.Cu")
